Commit message: added robot localization and madwick filter. robot localization runs only at 10Hz?

File: urdf/robot.urdf.xacro (robot description, xacro)
@@ -104,5 +104,5 @@
 <!-- Velodyne -->
 <xacro:include filename="$(find velodyne_description)/urdf/VLP-16.urdf.xacro"/>
-<xacro:VLP-16 parent="base_link" name="velodyne" topic="velodyne/points" organize_cloud="true" hz="15" samples="440" gpu="false">
+<xacro:VLP-16 parent="base_link" name="velodyne" topic="points" organize_cloud="true" hz="15" samples="440" gpu="false">
     <origin xyz="0 0 0.4" rpy="0.0 0.0 0.0" />
 </xacro:VLP-16>
@@ -122,35 +122,96 @@
     <parent link="base_link" />
     <child link="imu" />
-    <origin xyz="${imu_offset_x} ${imu_offset_y} ${imu_offset_z}" rpy="${M_PI} 0 ${M_PI/2.0}" />
+    <!-- <origin xyz="${imu_offset_x} ${imu_offset_y} ${imu_offset_z}" rpy="${M_PI} 0 ${M_PI/2.0}" /> -->
+    <origin xyz="${imu_offset_x} ${imu_offset_y} ${imu_offset_z}" rpy="0 0 0" />
 </joint>
-<!-- inertial measurement unit for gazebo -->
-<gazebo>
-    <plugin name="imu_controller" filename="libgazebo_ros_imu.so">
-    <alwaysOn>true</alwaysOn>
-    <updateRate>100.0</updateRate>
-    <bodyName>imu</bodyName>
-    <topicName>imu/data</topicName>
-    <serviceName>/default_imu</serviceName>
-    <gaussianNoise>${imu_stdev*imu_stdev}</gaussianNoise>
-    <xyzOffsets>0 0 0</xyzOffsets>
-    <rpyOffsets>0 0 0</rpyOffsets>
-    <interface:position name="imu_position"/>
+<gazebo reference="imu">
+    <sensor name="imu" type="imu">
+    <imu>
+        <angular_velocity>
+        <x>
+            <noise type="gaussian">
+            <mean>0.0</mean>
+            <stddev>${imu_stdev}</stddev>
+            </noise>
+        </x>
+        <y>
+            <noise type="gaussian">
+            <mean>0.0</mean>
+            <stddev>${imu_stdev}</stddev>
+            </noise>
+        </y>
+        <z>
+            <noise type="gaussian">
+            <mean>0.0</mean>
+            <stddev>${imu_stdev}</stddev>
+            </noise>
+        </z>
+        </angular_velocity>
+        <linear_acceleration>
+        <x>
+            <noise type="gaussian">
+            <mean>0.0</mean>
+            <stddev>${imu_stdev}</stddev>
+            </noise>
+        </x>
+        <y>
+            <noise type="gaussian">
+            <mean>0.0</mean>
+            <stddev>${imu_stdev}</stddev>
+            </noise>
+        </y>
+        <z>
+            <noise type="gaussian">
+            <mean>0.0</mean>
+            <stddev>${imu_stdev}</stddev>
+            </noise>
+        </z>
+        </linear_acceleration>
+    </imu>
+    <always_on>true</always_on>
+    <update_rate>100.0</update_rate>
+        <plugin name="imu_plugin" filename="libgazebo_ros_imu_sensor.so">
+        <initial_orientation_as_reference>false</initial_orientation_as_reference>
+        <ros>
+            <remapping>~/out:=/imu/data_raw</remapping>
+        </ros>
+        <frame_name>imu</frame_name>
     </plugin>
+    </sensor>
 </gazebo>
 <gazebo>
-    <plugin name="gazebo_ros_control" filename="libgazebo_ros_control.so">
-    </plugin>
-</gazebo>
-<!-- publish ground truth for pose of base_footprint -->
-<gazebo>
-    <plugin name="base_footprint_controller" filename="libgazebo_ros_p3d.so">
-    <alwaysOn>true</alwaysOn>
-    <updateRate>30.0</updateRate>
-    <bodyName>base_footprint</bodyName>
-    <topicName>base_footprint_pose_ground_truth</topicName>
-    <gaussianNoise>0.0</gaussianNoise>
-    <frameName>map</frameName>
-    <interface:position name="base_footprint_p3d_position_iface" />
-    </plugin>
+  <plugin name='skid_steer_drive' filename='libgazebo_ros_diff_drive.so'>
+    <!-- <ros>
+        <namespace>/demo</namespace>
+        <argument>cmd_vel:=cmd_demo</argument>
+        <argument>odom:=odom_demo</argument>
+    </ros> -->
+    <update_rate>100.0</update_rate>
+    <num_wheel_pairs>2</num_wheel_pairs>
+    <!-- wheels0 -->
+    <left_joint>left_front_wheel</left_joint>
+    <right_joint>right_front_wheel</right_joint>
+    <!-- wheels1-->
+    <left_joint>left_rear_wheel</left_joint>
+    <right_joint>right_rear_wheel</right_joint>
+    <!-- kinematics -->
+    <wheel_separation>${axis_length}</wheel_separation>
+    <wheel_separation>${axis_length}</wheel_separation>
+    <wheel_diameter>${2*wheel_radius}</wheel_diameter>
+    <wheel_diameter>${2*wheel_radius}</wheel_diameter>
+    <!-- limits -->
+    <max_wheel_torque>5000</max_wheel_torque>
+    <max_wheel_acceleration>3.0</max_wheel_acceleration>
+    <!-- Convariance -->
+    <covariance_x>0.001</covariance_x>
+    <covariance_y>0.001</covariance_y>
+    <covariance_yaw>0.001</covariance_yaw>
+    <!-- output -->
+    <publish_odom>true</publish_odom>
+    <publish_odom_tf>false</publish_odom_tf>
+    <publish_wheel_tf>true</publish_wheel_tf>
+    <odometry_frame>odom</odometry_frame>
+    <robot_base_frame>base_footprint</robot_base_frame>
+  </plugin>
 </gazebo>
 </robot>

Commit message: added text substitution

File: urdf/robot.urdf.xacro (robot description, xacro)
@@ -103,8 +103,74 @@
 </joint>
 <!-- Velodyne -->
-<xacro:include filename="$(find velodyne_description)/urdf/VLP-16.urdf.xacro"/>
-<xacro:VLP-16 parent="base_link" name="velodyne" topic="points" organize_cloud="true" hz="15" samples="440" gpu="false">
+<link name="velodyne">
+    <inertial>
+        <mass value="0.83"/>
+        <origin xyz="0 0 0.03585"/>
+        <inertia ixx="${(0.83 * (3.0*0.0516*0.0516 + 0.0717*0.0717)) / 12.0}" ixy="0" ixz="0"
+            iyy="${(0.83 * (3.0*0.0516*0.0516 + 0.0717*0.0717)) / 12.0}" iyz="0"
+            izz="${0.5 * 0.83 * (0.0516*0.0516)}"/>
+    </inertial>
+    <visual>
+        <origin rpy="0 0 0" xyz="0 0 0.03585"/>
+        <geometry>
+            <cylinder radius="0.0516" length="0.0717"/>
+        </geometry>
+    </visual>
+    <collision>
+        <origin rpy="0 0 0" xyz="0 0 0.03585"/>
+        <geometry>
+            <cylinder radius="0.0516" length="0.0717"/>
+        </geometry>
+    </collision>
+</link>
+<joint name="velodyne_to_base_joint" type="fixed">
+    <parent link="base_link" />
+    <child link="velodyne" />
     <origin xyz="0 0 0.4" rpy="0.0 0.0 0.0" />
-</xacro:VLP-16>
+</joint>
+<gazebo reference="velodyne">
+<sensor type="ray" name="velodyne-vlp16">
+    <pose>0 0 0 0 0 0</pose>
+    <visualize>false</visualize>
+    <update_rate>20</update_rate>
+    <ray>
+    <scan>
+        <horizontal>
+        <samples>440</samples>
+        <resolution>1</resolution>
+        <min_angle>-${M_PI}</min_angle>
+        <max_angle>${M_PI}</max_angle>
+        </horizontal>
+        <vertical>
+        <samples>16</samples>
+        <resolution>1</resolution>
+        <min_angle>-${M_PI*15.0/180.0}</min_angle>
+        <max_angle> ${M_PI*15.0/180.0}</max_angle>
+        </vertical>
+    </scan>
+    <range>
+        <min>0.3</min>
+        <max>130.0</max>
+        <resolution>0.001</resolution>
+    </range>
+    <noise>
+        <type>gaussian</type>
+        <mean>0.0</mean>
+        <stddev>0.0</stddev>
+    </noise>
+    </ray>
+    <plugin name="gazebo_ros_laser_controller" filename="libgazebo_ros_velodyne_laser.so">
+        <ros>
+            <namespace>/velodyne</namespace>
+            <remapping>~/out:=points</remapping>
+        </ros>
+        <frame_name>velodyne</frame_name>
+        <organize_cloud>true</organize_cloud>
+        <min_range>0.9</min_range>
+        <max_range>130.0</max_range>
+        <gaussian_noise>0.008</gaussian_noise>
+    </plugin>
+</sensor>
+</gazebo>
 <!-- IMU -->
 <link name="imu">
