Commit message: examples converted to new gazebo. not tested with rmcl

File: rmcl_sim/urdf/wheel.urdf.xacro (robot description, xacro)
@@ -25,6 +25,4 @@
             <mu1 value="1.0"/>
             <mu2 value="1.0"/>
-            <kp value="10000000.0" />
-            <kd value="1.0" />
             <fdir1 value="1 0 0"/>
             <material>Gazebo/DarkGrey</material>
@@ -36,14 +34,4 @@
             <axis xyz="0 1 0" rpy="0 0 0" />
         </joint>
-        <transmission name="${name}_trans" type="SimpleTransmission">
-            <type>transmission_interface/SimpleTransmission</type>
-            <actuator name="${name}_motor">
-                <mechanicalReduction>7</mechanicalReduction>
-                <hardwareInterface>VelocityJointInterface</hardwareInterface>
-            </actuator>
-            <joint name="${name}">
-                <hardwareInterface>hardware_interface/VelocityJointInterface</hardwareInterface>
-            </joint>
-        </transmission>
     </xacro:macro>
 </robot>
